File: pico_synth_sandbox.kicad_sch (KiCad schematic)
At the start: 44 parts, among them J1 UART0, J2 LINEOUT, SW1 RotaryEncoder_Switch, SW2 RESET, U1 Pico

Commit message: Revision 2 of schematic and pcb.
Parts:
- removed C1: 220uF, Capacitor_THT:CP_Radial_D5.0mm_P2.00mm, symbol Device:C_Polarized_Small
- removed J1: UART0, Connector_PinHeader_2.54mm:PinHeader_1x03_P2.54mm_Vertical, symbol Connector:Conn_01x03_Pin
- removed J2: LINEOUT, Connector_Audio:Jack_3.5mm_CUI_SJ1-3525N_Horizontal, symbol Connector_Audio:AudioJack3_SwitchTR
- removed JP1: PDMDAT, Jumper:SolderJumper-3_P1.3mm_Bridged12_RoundedPad1.0x1.5mm, symbol Jumper:SolderJumper_3_Bridged12
- removed JP2: PDMCLK, Jumper:SolderJumper-3_P1.3mm_Bridged12_RoundedPad1.0x1.5mm, symbol Jumper:SolderJumper_3_Bridged12
- removed JP3: I2SPWML, Jumper:SolderJumper-3_P1.3mm_Bridged12_RoundedPad1.0x1.5mm, symbol Jumper:SolderJumper_3_Bridged12
- removed JP4: I2SPWMR, Jumper:SolderJumper-3_P1.3mm_Bridged12_RoundedPad1.0x1.5mm, symbol Jumper:SolderJumper_3_Bridged12
- removed JP5: ALJP, Jumper:SolderJumper-3_P1.3mm_Bridged12_RoundedPad1.0x1.5mm, symbol Jumper:SolderJumper_3_Bridged12
- removed JP6: ARJP, Jumper:SolderJumper-3_P1.3mm_Bridged12_RoundedPad1.0x1.5mm, symbol Jumper:SolderJumper_3_Bridged12
- removed LS1: Speaker, Connector_JST:JST_GH_SM02B-GHS-TB_1x02-1MP_P1.25mm_Horizontal, symbol Device:Speaker
- removed R1, R10, R11, R12, R2, R3, R4, R5, R6, R7, R8, R9: 1M, Resistor_SMD:R_0805_2012Metric_Pad1.20x1.40mm_HandSolder, symbol Device:R_Small
- removed R13, R14: 10k, Resistor_THT:R_Axial_DIN0207_L6.3mm_D2.5mm_P7.62mm_Horizontal, symbol Device:R_Small
- removed RV2: 100k, Potentiometer_THT:Potentiometer_Alpha_RD902F-40-00D_Dual_Vertical, symbol Device:R_Potentiometer_Dual
- removed SW2: RESET, Button_Switch_SMD:SW_Push_1P1T_NO_6x6mm_H9.5mm, symbol Switch:SW_Push
- removed TP10: A, Capacitive_Keys:CapKeysWhiteMiddle, symbol Connector:TestPoint
- removed TP11: A#/Bb, Capacitive_Keys:CapKeysBlack, symbol Connector:TestPoint
- removed TP12: B, Capacitive_Keys:CapKeysWhiteRight, symbol Connector:TestPoint
- removed TP13, TP14: TestPoint, TestPoint:TestPoint_Pad_D2.0mm, symbol Connector:TestPoint
- removed TP4: D#/Eb, Capacitive_Keys:CapKeysBlack, symbol Connector:TestPoint
- removed TP5: E, Capacitive_Keys:CapKeysWhiteRight, symbol Connector:TestPoint
- removed TP6: F, Capacitive_Keys:CapKeysWhiteLeft, symbol Connector:TestPoint
- removed TP7: F#/Gb, Capacitive_Keys:CapKeysBlack, symbol Connector:TestPoint
- removed TP8: G, Capacitive_Keys:CapKeysWhiteMiddle, symbol Connector:TestPoint
- removed TP9: G#/Ab, Capacitive_Keys:CapKeysBlack, symbol Connector:TestPoint
- added C10: 2.2uF, Capacitor_SMD:C_0805_2012Metric_Pad1.18x1.45mm_HandSolder, symbol Device:C_Small
- added C3: 10uF, Capacitor_SMD:C_0805_2012Metric_Pad1.18x1.45mm_HandSolder, symbol Device:C_Small
- added C4: 0.1uF, Capacitor_SMD:C_0805_2012Metric_Pad1.18x1.45mm_HandSolder, symbol Device:C_Small
- added C8: 470pF, Capacitor_SMD:C_0805_2012Metric_Pad1.18x1.45mm_HandSolder, symbol Device:C_Small
- added FB1: EFI_GNDA, Resistor_SMD:R_0805_2012Metric_Pad1.20x1.40mm_HandSolder, symbol Device:FerriteBead_Small
- added H1, H2, H3, H4: MountingHole_Pad, MountingHole:MountingHole_2.5mm_Pad, symbol Mechanical:MountingHole_Pad
- added J1: Micro_SD_Card_Det2, Connector_Card:microSD_HC_Hirose_DM3D-SF, symbol Connector:Micro_SD_Card_Det2
- added RN1, RN2: 47k, Resistor_SMD:R_Array_Convex_4x1206, symbol Device:R_Pack04
- added SW2: RotaryEncoder_Switch, Rotary_Encoder:RotaryEncoder_Alps_EC11E-Switch_Vertical_H20mm, symbol Device:RotaryEncoder_Switch
- added SW3: PWR_EN, pico_synth_sandbox:MK-23D38, symbol Switch:SW_DP3T
- added U2: MIC5219-3.3YM5, Package_TO_SOT_SMD:SOT-23-5, symbol Regulator_Linear:MIC5219-3.3YM5
- TP1: value C -> SD_DAT1; footprint Capacitive_Keys:CapKeysWhiteLeft -> TestPoint:TestPoint_Pad_D2.0mm
- TP2: value C#/Db -> SD_DAT2; footprint Capacitive_Keys:CapKeysBlack -> TestPoint:TestPoint_Pad_D2.0mm
- TP3: value D -> SD_DET; footprint Capacitive_Keys:CapKeysWhiteMiddle -> TestPoint:TestPoint_Pad_D2.0mm
- U1: footprint MCU_RaspberryPi_and_Boards:RPi_Pico_SMD_TH -> pico_synth_sandbox:RPi_Pico_SMD_TH_BS
Connections:
- net TPAD10 is gone; now on net ENC1SW: U1.17 (GPIO13)
- net TPAD4 is gone; now on net 1602RS: U1.10 (GPIO7)
- net TPAD8 is gone; now on net ENC1A: U1.15 (GPIO11)
- net TPAD9 is gone; now on net ENC1B: U1.16 (GPIO12)
- net +3.3V: now also C3.1, C4.1, J1.4 (VDD), RN1.5 (R4.2), RN1.6 (R3.2), RN1.7 (R2.2), RN1.8 (R1.2), RN2.5 (R4.2), RN2.6 (R3.2), RN2.7 (R2.2), RN2.8 (R1.2)
- net +5V: now also RV1.3, SW3.3; no longer RV1.1
- net 1602EN: now also U1.9 (GPIO6); no longer U1.27 (GPIO21)
- net 1602RS: no longer U1.26 (GPIO20)
- net 3V3_EN: now also SW3.7, U2.3 (EN)
- net GND: now also RV1.1, C10.2, C3.2, C4.2, C8.2, FB1.1, H1.1, H2.1, H3.1, H4.1, J1.11 (SHIELD), J1.6 (VSS), SW2.C, SW2.S2, SW3.8, U2.2 (GND); no longer RV1.3
- net GNDA: now also FB1.2
- net VSYS: now also SW3.1, U2.1 (IN)
- net UART_RX: now reaches U1.7 (GPIO5)
- net ENC2A: now reaches U1.21 (GPIO16)
- net ENC2A: now also SW2.A
- net ENC2B: now reaches U1.22 (GPIO17)
- net ENC2B: now also SW2.B
- net UART_TX: now reaches U1.6 (GPIO4)
- net ENCA renamed ENC1A
- net ENC1A: no longer U1.1 (GPIO0)
- net ENCB renamed ENC1B
- net ENC1B: no longer U1.2 (GPIO1)
- net I2SDAT renamed ENC2SW
- net ENC2SW: now also SW2.S1
- net SWA renamed ENC1SW
- net ENC1SW: no longer U1.4 (GPIO2)
- net TPAD1: no longer names the net of TP1.1
- net TPAD1: now also J1.8 (DAT1), RN2.1 (R1.1); no longer U1.25 (GPIO19)
- net TPAD11 renamed TTP_SDO
- net TPAD12 renamed TTP_SCL
- net TPAD2: no longer names the net of TP2.1
- net TPAD2: now also J1.1 (DAT2), RN1.1 (R1.1); no longer U1.5 (GPIO3)
- net TPAD3: no longer names the net of TP3.1
- net TPAD3: now also J1.10 (DET_A), RN2.3 (R3.1); no longer U1.9 (GPIO6)
- net TPAD5 renamed ADC_I2SCLK
- net TPAD6 renamed ADC_I2SWS
- net TPAD7 renamed ADC_I2SDAT
- new net: C8.1, U2.4 (BP)
- new net +3.3VA: C10.1, U2.5 (OUT)
- new net DAC_I2SCLK: U1.25 (GPIO19)
- new net DAC_I2SDAT: U1.27 (GPIO21)
- new net DAC_I2SWS: U1.26 (GPIO20)
- new net SPI_CS: J1.2 (DAT3/CD), RN1.2 (R2.1), U1.2 (GPIO1)
- new net SPI_RX: J1.7 (DAT0), RN2.2 (R2.1), U1.1 (GPIO0)
- new net SPI_SCK: J1.5 (CLK), RN2.4 (R4.1), U1.4 (GPIO2)
- new net SPI_TX: J1.3 (CMD), RN1.3 (R3.1), U1.5 (GPIO3)
- no-connect marks 6 -> 7
Other:
- sheet Audio Input renamed I2S ADC
- sheet I2S Audio renamed I2S DAC
- removed sheet PWM Audio
- added sheet Audio Output (audio_out.kicad_sch)
- added sheet Touch Keyboard (keyboard.kicad_sch)
- sheet I2S ADC: file audio_in.kicad_sch -> i2s_adc.kicad_sch
- sheet I2S DAC: file i2s_audio.kicad_sch -> i2s_dac.kicad_sch
- note added: "3.3v Analog Power Supply"
- note added: "Encoders"
- note added: "MCU"
- note added: "Micro SD Card"
- note added: "Power Enable"
- note removed: "Audio Output"
- note removed: "Capacitive Keyboard"
- title: pico_synth_sandbox -> pico_synth_sandbox - MCU
- moved on the sheet: DS1, SW1, U1
