File: pico_synth_sandbox.kicad_sch (KiCad schematic)
At the start: 22 parts, among them J1 Micro_SD_Card_Det2, SW1 RotaryEncoder_Switch, SW2 RotaryEncoder_Switch, SW3 PWR_EN, U1 Pico, U2 MIC5219-3.3YM5

Commit message: Fixed character lcd data pin references.
Parts:
- renumbered C8 to C1, C10 to C2
Connections:
- net 1602D4: now also DS1.11 (D4), U1.29 (GPIO22); no longer DS1.14 (D7), U1.34 (GPIO28_ADC2)
- net 1602D5: now also DS1.12 (D5), U1.31 (GPIO26_ADC0); no longer DS1.13 (D6), U1.32 (GPIO27_ADC1)
- net 1602D6: now also DS1.13 (D6), U1.32 (GPIO27_ADC1); no longer DS1.12 (D5), U1.31 (GPIO26_ADC0)
- net 1602D7: now also DS1.14 (D7), U1.34 (GPIO28_ADC2); no longer DS1.11 (D4), U1.29 (GPIO22)
