File: i2s_adc.kicad_sch (KiCad schematic)
At the start: 28 parts, among them J2 LINEIN, U4 PCM1860DBTR

Commit message: Minor update to ADC connection.
Parts:
- R3: value 100k -> 1k
Connections:
- net at U4.19 (INT): no longer RN4.4 (R4.1)
- no-connect marks 2 -> 3
Other:
- note added: "Not sure about the implementation of INT here. Maybe GND it?"
Changed lines of the file:
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@@
   (no_connect (at 118.11 129.54))
   (no_connect (at 118.11 132.08))
+  (no_connect (at 148.59 106.68))
   (wire (pts (xy 43.18 180.34) (xy 43.18 177.8))
     (stroke (width 0) (type default))
@@
     (stroke (width 0) (type default))
   )
-  (wire (pts (xy 148.59 106.68) (xy 157.48 106.68))
-    (stroke (width 0) (type default))
-  )
   (wire (pts (xy 153.67 111.76) (xy 165.1 111.76))
     (stroke (width 0) (type default))
@@
   )
   (wire (pts (xy 95.25 116.84) (xy 106.68 116.84))
-    (stroke (width 0) (type default))
-  )
-  (wire (pts (xy 157.48 106.68) (xy 157.48 130.81))
     (stroke (width 0) (type default))
   )
@@
   (text "Line Input" (at 19.05 22.86 0)
     (effects (font (size 2.54 2.54) (thickness 0.508) bold) (justify left bottom))
+  )
+  (text "Not sure about the implementation of INT here. Maybe GND it?"
+    (at 151.13 107.95 0)
+    (effects (font (size 1.27 1.27)) (justify left bottom))
   )
   (text "Power Filtering" (at 39.37 158.75 0)
@@
       (effects (font (size 1.27 1.27)) (justify left))
     )
-    (property "Value" "100k" (at 46.99 30.48 0)
+    (property "Value" "1k" (at 46.99 30.48 0)
       (effects (font (size 1.27 1.27)) (justify left))
     )
