File: i2s_adc.kicad_sch (KiCad schematic)
At the start: 28 parts, among them J2 LINEIN, U4 PCM1860DBTR

Commit message: Various minor schematic updates.
Parts:
- renumbered RN3 to RN5, TP4 to TP5
Changed lines of the file:
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@@
   (symbol (lib_id "power:+3.3V") (at 130.81 76.2 0) (unit 1)
     (in_bom yes) (on_board yes) (dnp no)
-    (property "Reference" "#PWR09" (at 130.81 80.01 0)
+    (property "Reference" "#PWR071" (at 130.81 80.01 0)
       (effects (font (size 1.27 1.27)) hide)
     )
@@
     (instances
       (project "pico_synth_sandbox"
-        (path "/bfc01388-33ce-4b1a-9d2f-82d750172e5a"
-          (reference "#PWR09") (unit 1)
-        )
-        (path "/bfc01388-33ce-4b1a-9d2f-82d750172e5a/f0d7f11b-6ebd-4c2b-8e52-e814f3b2f284"
-          (reference "#PWR034") (unit 1)
-        )
         (path "/bfc01388-33ce-4b1a-9d2f-82d750172e5a/93632245-6c20-4ae6-b62e-7dbbebc316d1"
           (reference "#PWR071") (unit 1)
@@
   (symbol (lib_id "power:+3.3VA") (at 138.43 76.2 0) (unit 1)
     (in_bom yes) (on_board yes) (dnp no)
-    (property "Reference" "#PWR036" (at 138.43 80.01 0)
+    (property "Reference" "#PWR073" (at 138.43 80.01 0)
       (effects (font (size 1.27 1.27)) hide)
     )
@@
     (instances
       (project "pico_synth_sandbox"
-        (path "/bfc01388-33ce-4b1a-9d2f-82d750172e5a/f0d7f11b-6ebd-4c2b-8e52-e814f3b2f284"
-          (reference "#PWR036") (unit 1)
-        )
         (path "/bfc01388-33ce-4b1a-9d2f-82d750172e5a/93632245-6c20-4ae6-b62e-7dbbebc316d1"
           (reference "#PWR073") (unit 1)
@@
   (symbol (lib_id "power:+3.3VA") (at 48.26 24.13 0) (unit 1)
     (in_bom yes) (on_board yes) (dnp no)
-    (property "Reference" "#PWR036" (at 48.26 27.94 0)
+    (property "Reference" "#PWR063" (at 48.26 27.94 0)
       (effects (font (size 1.27 1.27)) hide)
     )
@@
     (instances
       (project "pico_synth_sandbox"
-        (path "/bfc01388-33ce-4b1a-9d2f-82d750172e5a/f0d7f11b-6ebd-4c2b-8e52-e814f3b2f284"
-          (reference "#PWR036") (unit 1)
-        )
         (path "/bfc01388-33ce-4b1a-9d2f-82d750172e5a/93632245-6c20-4ae6-b62e-7dbbebc316d1"
           (reference "#PWR063") (unit 1)
@@
   (symbol (lib_id "Connector:TestPoint") (at 176.53 101.6 270) (mirror x) (unit 1)
     (in_bom yes) (on_board yes) (dnp no)
-    (property "Reference" "TP4" (at 181.61 101.6 90)
+    (property "Reference" "TP5" (at 181.61 101.6 90)
       (effects (font (size 1.27 1.27)) (justify left))
     )
@@
     (instances
       (project "pico_synth_sandbox"
-        (path "/bfc01388-33ce-4b1a-9d2f-82d750172e5a/f0d7f11b-6ebd-4c2b-8e52-e814f3b2f284"
-          (reference "TP4") (unit 1)
-        )
         (path "/bfc01388-33ce-4b1a-9d2f-82d750172e5a/93632245-6c20-4ae6-b62e-7dbbebc316d1"
           (reference "TP5") (unit 1)
@@
   (symbol (lib_id "power:+3.3VA") (at 68.58 167.64 0) (unit 1)
     (in_bom yes) (on_board yes) (dnp no)
-    (property "Reference" "#PWR036" (at 68.58 171.45 0)
+    (property "Reference" "#PWR065" (at 68.58 171.45 0)
       (effects (font (size 1.27 1.27)) hide)
     )
@@
     (instances
       (project "pico_synth_sandbox"
-        (path "/bfc01388-33ce-4b1a-9d2f-82d750172e5a/f0d7f11b-6ebd-4c2b-8e52-e814f3b2f284"
-          (reference "#PWR036") (unit 1)
-        )
         (path "/bfc01388-33ce-4b1a-9d2f-82d750172e5a/93632245-6c20-4ae6-b62e-7dbbebc316d1"
           (reference "#PWR065") (unit 1)
@@
   (symbol (lib_id "power:+3.3V") (at 165.1 109.22 0) (unit 1)
     (in_bom yes) (on_board yes) (dnp no)
-    (property "Reference" "#PWR09" (at 165.1 113.03 0)
+    (property "Reference" "#PWR076" (at 165.1 113.03 0)
       (effects (font (size 1.27 1.27)) hide)
     )
@@
     (instances
       (project "pico_synth_sandbox"
-        (path "/bfc01388-33ce-4b1a-9d2f-82d750172e5a"
-          (reference "#PWR09") (unit 1)
-        )
-        (path "/bfc01388-33ce-4b1a-9d2f-82d750172e5a/f0d7f11b-6ebd-4c2b-8e52-e814f3b2f284"
-          (reference "#PWR034") (unit 1)
-        )
         (path "/bfc01388-33ce-4b1a-9d2f-82d750172e5a/93632245-6c20-4ae6-b62e-7dbbebc316d1"
           (reference "#PWR076") (unit 1)
@@
   (symbol (lib_id "power:+3.3VA") (at 232.41 39.37 0) (unit 1)
     (in_bom yes) (on_board yes) (dnp no)
-    (property "Reference" "#PWR036" (at 232.41 43.18 0)
+    (property "Reference" "#PWR079" (at 232.41 43.18 0)
       (effects (font (size 1.27 1.27)) hide)
     )
@@
     (instances
       (project "pico_synth_sandbox"
-        (path "/bfc01388-33ce-4b1a-9d2f-82d750172e5a/f0d7f11b-6ebd-4c2b-8e52-e814f3b2f284"
-          (reference "#PWR036") (unit 1)
-        )
         (path "/bfc01388-33ce-4b1a-9d2f-82d750172e5a/93632245-6c20-4ae6-b62e-7dbbebc316d1"
           (reference "#PWR079") (unit 1)
@@
   (symbol (lib_id "Device:R_Pack04") (at 165.1 99.06 270) (unit 1)
     (in_bom yes) (on_board yes) (dnp no)
-    (property "Reference" "RN3" (at 165.1 88.9 90)
+    (property "Reference" "RN5" (at 165.1 88.9 90)
       (effects (font (size 1.27 1.27)))
     )
@@
     (instances
       (project "pico_synth_sandbox"
-        (path "/bfc01388-33ce-4b1a-9d2f-82d750172e5a/f0d7f11b-6ebd-4c2b-8e52-e814f3b2f284"
-          (reference "RN3") (unit 1)
-        )
         (path "/bfc01388-33ce-4b1a-9d2f-82d750172e5a/93632245-6c20-4ae6-b62e-7dbbebc316d1"
           (reference "RN5") (unit 1)
@@
   (symbol (lib_id "power:+3.3VA") (at 180.34 39.37 0) (unit 1)
     (in_bom yes) (on_board yes) (dnp no)
-    (property "Reference" "#PWR036" (at 180.34 43.18 0)
+    (property "Reference" "#PWR077" (at 180.34 43.18 0)
       (effects (font (size 1.27 1.27)) hide)
     )
@@
     (instances
       (project "pico_synth_sandbox"
-        (path "/bfc01388-33ce-4b1a-9d2f-82d750172e5a/f0d7f11b-6ebd-4c2b-8e52-e814f3b2f284"
-          (reference "#PWR036") (unit 1)
-        )
         (path "/bfc01388-33ce-4b1a-9d2f-82d750172e5a/93632245-6c20-4ae6-b62e-7dbbebc316d1"
           (reference "#PWR077") (unit 1)
@@
   (symbol (lib_id "power:+3.3V") (at 45.72 167.64 0) (unit 1)
     (in_bom yes) (on_board yes) (dnp no)
-    (property "Reference" "#PWR09" (at 45.72 171.45 0)
+    (property "Reference" "#PWR061" (at 45.72 171.45 0)
       (effects (font (size 1.27 1.27)) hide)
     )
@@
     (instances
       (project "pico_synth_sandbox"
-        (path "/bfc01388-33ce-4b1a-9d2f-82d750172e5a"
-          (reference "#PWR09") (unit 1)
-        )
-        (path "/bfc01388-33ce-4b1a-9d2f-82d750172e5a/f0d7f11b-6ebd-4c2b-8e52-e814f3b2f284"
-          (reference "#PWR034") (unit 1)
-        )
         (path "/bfc01388-33ce-4b1a-9d2f-82d750172e5a/93632245-6c20-4ae6-b62e-7dbbebc316d1"
           (reference "#PWR061") (unit 1)
