File: audio_out.kicad_sch (KiCad schematic)
At the start: 44 parts, among them J10 HPOUT, J10 LINEOUT, J4 SPKRL, J5 SPKRR, Q1 BSS138, Q2 BSS138, U5 PAM8019

Commit message: Various minor schematic updates.
Parts:
- renumbered C28 to C39, C29 to C40, C29 to C41, C29 to C42, FB1 to FB2, FB2 to FB3, FB1 to FB4, FB2 to FB5, J10 to J3, J10 to J6, RV2 to RV3, TP13 to TP6, TP14 to TP7, TP13 to TP8, TP14 to TP9
Changed lines of the file:
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@@
   (symbol (lib_id "Connector:TestPoint") (at 165.1 96.52 0) (mirror x) (unit 1)
     (in_bom yes) (on_board yes) (dnp no)
-    (property "Reference" "TP14" (at 163.83 99.06 0)
+    (property "Reference" "TP9" (at 163.83 99.06 0)
       (effects (font (size 1.27 1.27)) (justify right))
     )
@@
     (instances
       (project "pico_synth_sandbox"
-        (path "/bfc01388-33ce-4b1a-9d2f-82d750172e5a"
-          (reference "TP14") (unit 1)
-        )
         (path "/bfc01388-33ce-4b1a-9d2f-82d750172e5a/95658688-f49d-4f25-a927-5c37230192e0"
           (reference "TP9") (unit 1)
@@
   (symbol (lib_id "Device:FerriteBead_Small") (at 127 96.52 270) (unit 1)
     (in_bom yes) (on_board yes) (dnp no)
-    (property "Reference" "FB2" (at 129.54 99.06 90)
+    (property "Reference" "FB3" (at 129.54 99.06 90)
       (effects (font (size 1.27 1.27)))
     )
@@
     (instances
       (project "pico_synth_sandbox"
-        (path "/bfc01388-33ce-4b1a-9d2f-82d750172e5a"
-          (reference "FB2") (unit 1)
-        )
         (path "/bfc01388-33ce-4b1a-9d2f-82d750172e5a/95658688-f49d-4f25-a927-5c37230192e0"
           (reference "FB3") (unit 1)
@@
   (symbol (lib_id "Connector_Audio:AudioJack4_SwitchT1") (at 109.22 165.1 180) (unit 1)
     (in_bom yes) (on_board yes) (dnp no)
-    (property "Reference" "J10" (at 119.38 161.925 0)
+    (property "Reference" "J3" (at 119.38 161.925 0)
       (effects (font (size 1.27 1.27)) (justify right))
     )
@@
     (instances
       (project "pico_synth_sandbox"
-        (path "/bfc01388-33ce-4b1a-9d2f-82d750172e5a/93632245-6c20-4ae6-b62e-7dbbebc316d1"
-          (reference "J10") (unit 1)
-        )
         (path "/bfc01388-33ce-4b1a-9d2f-82d750172e5a/95658688-f49d-4f25-a927-5c37230192e0"
           (reference "J3") (unit 1)
@@
   (symbol (lib_id "Device:FerriteBead_Small") (at 130.81 85.09 270) (unit 1)
     (in_bom yes) (on_board yes) (dnp no)
-    (property "Reference" "FB2" (at 133.35 87.63 90)
+    (property "Reference" "FB5" (at 133.35 87.63 90)
       (effects (font (size 1.27 1.27)))
     )
@@
     (instances
       (project "pico_synth_sandbox"
-        (path "/bfc01388-33ce-4b1a-9d2f-82d750172e5a"
-          (reference "FB2") (unit 1)
-        )
         (path "/bfc01388-33ce-4b1a-9d2f-82d750172e5a/95658688-f49d-4f25-a927-5c37230192e0"
           (reference "FB5") (unit 1)
@@
   (symbol (lib_id "power:GNDA") (at 101.6 175.26 0) (mirror y) (unit 1)
     (in_bom yes) (on_board yes) (dnp no)
-    (property "Reference" "#PWR020" (at 101.6 181.61 0)
+    (property "Reference" "#PWR097" (at 101.6 181.61 0)
       (effects (font (size 1.27 1.27)) hide)
     )
@@
     (instances
       (project "pico_synth_sandbox"
-        (path "/bfc01388-33ce-4b1a-9d2f-82d750172e5a"
-          (reference "#PWR020") (unit 1)
-        )
         (path "/bfc01388-33ce-4b1a-9d2f-82d750172e5a/95658688-f49d-4f25-a927-5c37230192e0"
           (reference "#PWR097") (unit 1)
@@
   (symbol (lib_id "Connector:TestPoint") (at 165.1 82.55 0) (unit 1)
     (in_bom yes) (on_board yes) (dnp no)
-    (property "Reference" "TP13" (at 163.83 80.01 0)
+    (property "Reference" "TP6" (at 163.83 80.01 0)
       (effects (font (size 1.27 1.27)) (justify right))
     )
@@
     (instances
       (project "pico_synth_sandbox"
-        (path "/bfc01388-33ce-4b1a-9d2f-82d750172e5a"
-          (reference "TP13") (unit 1)
-        )
         (path "/bfc01388-33ce-4b1a-9d2f-82d750172e5a/95658688-f49d-4f25-a927-5c37230192e0"
           (reference "TP6") (unit 1)
@@
   (symbol (lib_id "Device:C_Small") (at 135.89 106.68 0) (mirror y) (unit 1)
     (in_bom yes) (on_board yes) (dnp no)
-    (property "Reference" "C28" (at 134.62 105.41 90)
+    (property "Reference" "C39" (at 134.62 105.41 90)
       (effects (font (size 1.27 1.27)) (justify left))
     )
@@
     (instances
       (project "pico_synth_sandbox"
-        (path "/bfc01388-33ce-4b1a-9d2f-82d750172e5a"
-          (reference "C28") (unit 1)
-        )
         (path "/bfc01388-33ce-4b1a-9d2f-82d750172e5a/95658688-f49d-4f25-a927-5c37230192e0"
           (reference "C39") (unit 1)
@@
   (symbol (lib_id "pico_synth_sandbox:RK10J12R0A0B") (at 48.26 67.31 0) (unit 1)
     (in_bom yes) (on_board yes) (dnp no)
-    (property "Reference" "RV2" (at 49.53 67.31 90)
+    (property "Reference" "RV3" (at 49.53 67.31 90)
       (effects (font (size 1.27 1.27)))
     )
@@
     (instances
       (project "pico_synth_sandbox"
-        (path "/bfc01388-33ce-4b1a-9d2f-82d750172e5a/93632245-6c20-4ae6-b62e-7dbbebc316d1"
-          (reference "RV2") (unit 1)
-        )
         (path "/bfc01388-33ce-4b1a-9d2f-82d750172e5a/95658688-f49d-4f25-a927-5c37230192e0"
           (reference "RV3") (unit 1)
@@
   (symbol (lib_id "Device:C_Small") (at 147.32 106.68 0) (unit 1)
     (in_bom yes) (on_board yes) (dnp no)
-    (property "Reference" "C29" (at 146.05 105.41 90)
+    (property "Reference" "C42" (at 146.05 105.41 90)
       (effects (font (size 1.27 1.27)) (justify left))
     )
@@
     (instances
       (project "pico_synth_sandbox"
-        (path "/bfc01388-33ce-4b1a-9d2f-82d750172e5a"
-          (reference "C29") (unit 1)
-        )
         (path "/bfc01388-33ce-4b1a-9d2f-82d750172e5a/95658688-f49d-4f25-a927-5c37230192e0"
           (reference "C42") (unit 1)
@@
   (symbol (lib_id "Connector:TestPoint") (at 165.1 85.09 0) (mirror x) (unit 1)
     (in_bom yes) (on_board yes) (dnp no)
-    (property "Reference" "TP14" (at 163.83 87.63 0)
+    (property "Reference" "TP7" (at 163.83 87.63 0)
       (effects (font (size 1.27 1.27)) (justify right))
     )
@@
     (instances
       (project "pico_synth_sandbox"
-        (path "/bfc01388-33ce-4b1a-9d2f-82d750172e5a"
-          (reference "TP14") (unit 1)
-        )
         (path "/bfc01388-33ce-4b1a-9d2f-82d750172e5a/95658688-f49d-4f25-a927-5c37230192e0"
           (reference "TP7") (unit 1)
@@
   (symbol (lib_id "Device:FerriteBead_Small") (at 128.27 82.55 90) (unit 1)
     (in_bom yes) (on_board yes) (dnp no)
-    (property "Reference" "FB1" (at 130.81 80.01 90)
+    (property "Reference" "FB4" (at 130.81 80.01 90)
       (effects (font (size 1.27 1.27)))
     )
@@
     (instances
       (project "pico_synth_sandbox"
-        (path "/bfc01388-33ce-4b1a-9d2f-82d750172e5a"
-          (reference "FB1") (unit 1)
-        )
         (path "/bfc01388-33ce-4b1a-9d2f-82d750172e5a/95658688-f49d-4f25-a927-5c37230192e0"
           (reference "FB4") (unit 1)
@@
   (symbol (lib_id "Device:C_Small") (at 143.51 106.68 0) (unit 1)
     (in_bom yes) (on_board yes) (dnp no)
-    (property "Reference" "C29" (at 142.24 105.41 90)
+    (property "Reference" "C41" (at 142.24 105.41 90)
       (effects (font (size 1.27 1.27)) (justify left))
     )
@@
     (instances
       (project "pico_synth_sandbox"
-        (path "/bfc01388-33ce-4b1a-9d2f-82d750172e5a"
-          (reference "C29") (unit 1)
-        )
         (path "/bfc01388-33ce-4b1a-9d2f-82d750172e5a/95658688-f49d-4f25-a927-5c37230192e0"
           (reference "C41") (unit 1)
@@
   (symbol (lib_id "Device:FerriteBead_Small") (at 124.46 93.98 90) (unit 1)
     (in_bom yes) (on_board yes) (dnp no)
-    (property "Reference" "FB1" (at 127 91.44 90)
+    (property "Reference" "FB2" (at 127 91.44 90)
       (effects (font (size 1.27 1.27)))
     )
@@
     (instances
       (project "pico_synth_sandbox"
-        (path "/bfc01388-33ce-4b1a-9d2f-82d750172e5a"
-          (reference "FB1") (unit 1)
-        )
         (path "/bfc01388-33ce-4b1a-9d2f-82d750172e5a/95658688-f49d-4f25-a927-5c37230192e0"
           (reference "FB2") (unit 1)
@@
   (symbol (lib_id "Connector_Audio:AudioJack4_SwitchT1") (at 241.3 144.78 180) (unit 1)
     (in_bom yes) (on_board yes) (dnp no)
-    (property "Reference" "J10" (at 251.46 141.605 0)
+    (property "Reference" "J6" (at 251.46 141.605 0)
       (effects (font (size 1.27 1.27)) (justify right))
     )
@@
     (instances
       (project "pico_synth_sandbox"
-        (path "/bfc01388-33ce-4b1a-9d2f-82d750172e5a/93632245-6c20-4ae6-b62e-7dbbebc316d1"
-          (reference "J10") (unit 1)
-        )
         (path "/bfc01388-33ce-4b1a-9d2f-82d750172e5a/95658688-f49d-4f25-a927-5c37230192e0"
           (reference "J6") (unit 1)
@@
   (symbol (lib_id "Connector:TestPoint") (at 165.1 93.98 0) (unit 1)
     (in_bom yes) (on_board yes) (dnp no)
-    (property "Reference" "TP13" (at 163.83 91.44 0)
+    (property "Reference" "TP8" (at 163.83 91.44 0)
       (effects (font (size 1.27 1.27)) (justify right))
     )
@@
     (instances
       (project "pico_synth_sandbox"
-        (path "/bfc01388-33ce-4b1a-9d2f-82d750172e5a"
-          (reference "TP13") (unit 1)
-        )
         (path "/bfc01388-33ce-4b1a-9d2f-82d750172e5a/95658688-f49d-4f25-a927-5c37230192e0"
           (reference "TP8") (unit 1)
@@
   (symbol (lib_id "Device:C_Small") (at 139.7 106.68 0) (unit 1)
     (in_bom yes) (on_board yes) (dnp no)
-    (property "Reference" "C29" (at 138.43 105.41 90)
+    (property "Reference" "C40" (at 138.43 105.41 90)
       (effects (font (size 1.27 1.27)) (justify left))
     )
@@
     (instances
       (project "pico_synth_sandbox"
-        (path "/bfc01388-33ce-4b1a-9d2f-82d750172e5a"
-          (reference "C29") (unit 1)
-        )
         (path "/bfc01388-33ce-4b1a-9d2f-82d750172e5a/95658688-f49d-4f25-a927-5c37230192e0"
           (reference "C40") (unit 1)
