File: battery.kicad_sch (KiCad schematic)
At the start: 24 parts, among them Q1 BSS84, Q2 BSS84, Q2 MMBT3904, Q6 BSS84, Q7 BSS138, SW3 PWR_EN, U6 MCP73831-5-OT, U7 AP9101CK6

Commit message: Revision 2 of schematic and pcb.
Parts:
- removed JP14: 5V_PWR, Jumper:SolderJumper-2_P1.3mm_Open_RoundedPad1.0x1.5mm, symbol Jumper:SolderJumper_2_Open
- removed Q2: MMBT3904, Package_TO_SOT_SMD:SOT-23_Handsoldering, symbol Transistor_BJT:MMBT3904
- removed Q6: BSS84, Package_TO_SOT_SMD:SOT-23_Handsoldering, symbol Transistor_FET:BSS84
- removed R38, R39: 330, Resistor_SMD:R_0805_2012Metric_Pad1.20x1.40mm_HandSolder, symbol Device:R_Small
- removed R40: 4.7k, Resistor_SMD:R_0805_2012Metric_Pad1.20x1.40mm_HandSolder, symbol Device:R_Small
- removed SW3: PWR_EN, Button_Switch_THT:SW_CuK_OS102011MA1QN1_SPDT_Angled, symbol Switch:SW_SPST
- renumbered C23 to C43, C24 to C44, C25 to C45, D2 to D1, D3 to D2, Q1 to Q3, Q2 to Q4, R33 to R15, R34 to R16, R35 to R17, R36 to R18, R37 to R19
Other:
- title: pico_synth_sandbox -> pico_synth_sandbox - LiPo Battery Power & Charging

Commit message: Various minor schematic updates.
Parts:
- renumbered Q7 to Q5, Q7 to Q6
Changed lines of the file:
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@@
   (symbol (lib_id "Transistor_FET:BSS138") (at 191.77 82.55 270) (unit 1)
     (in_bom yes) (on_board yes) (dnp no) (fields_autoplaced)
-    (property "Reference" "Q7" (at 191.77 88.9 90)
+    (property "Reference" "Q5" (at 191.77 88.9 90)
       (effects (font (size 1.27 1.27)))
     )
@@
     (instances
       (project "pico_synth_sandbox"
-        (path "/bfc01388-33ce-4b1a-9d2f-82d750172e5a"
-          (reference "Q7") (unit 1)
-        )
         (path "/bfc01388-33ce-4b1a-9d2f-82d750172e5a/9c12b2ee-f811-4183-acdf-4598ef52f2ef"
           (reference "Q5") (unit 1)
@@
   (symbol (lib_id "Transistor_FET:BSS138") (at 205.74 82.55 90) (mirror x) (unit 1)
     (in_bom yes) (on_board yes) (dnp no)
-    (property "Reference" "Q7" (at 205.74 88.9 90)
+    (property "Reference" "Q6" (at 205.74 88.9 90)
       (effects (font (size 1.27 1.27)))
     )
@@
     (instances
       (project "pico_synth_sandbox"
-        (path "/bfc01388-33ce-4b1a-9d2f-82d750172e5a"
-          (reference "Q7") (unit 1)
-        )
         (path "/bfc01388-33ce-4b1a-9d2f-82d750172e5a/9c12b2ee-f811-4183-acdf-4598ef52f2ef"
           (reference "Q6") (unit 1)
