File: keyboard.kicad_sch (KiCad schematic)
At the start: 35 parts, among them U8 TTP229-BSF

Commit message: Various minor schematic updates.
Parts:
- renumbered TP1 to TP10, TP2 to TP11, TP3 to TP12, TP4 to TP13, TP5 to TP14, TP6 to TP15, TP7 to TP16, TP8 to TP17, TP9 to TP18, TP10 to TP19, TP11 to TP20, TP12 to TP21, TP13 to TP22, TP14 to TP23, TP15 to TP24, TP16 to TP25
Changed lines of the file:
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@@
   (symbol (lib_id "Connector:TestPoint") (at 149.86 50.8 0) (mirror y) (unit 1)
     (in_bom yes) (on_board yes) (dnp no)
-    (property "Reference" "TP11" (at 151.13 49.53 0)
+    (property "Reference" "TP20" (at 151.13 49.53 0)
       (effects (font (size 1.27 1.27)) (justify right))
     )
@@
     (instances
       (project "pico_synth_sandbox"
-        (path "/bfc01388-33ce-4b1a-9d2f-82d750172e5a"
-          (reference "TP11") (unit 1)
-        )
         (path "/bfc01388-33ce-4b1a-9d2f-82d750172e5a/c37b2c46-91dc-4067-923d-eccca1cbe357"
           (reference "TP20") (unit 1)
@@
   (symbol (lib_id "Connector:TestPoint") (at 157.48 41.91 0) (mirror y) (unit 1)
     (in_bom yes) (on_board yes) (dnp no)
-    (property "Reference" "TP12" (at 158.75 40.64 0)
+    (property "Reference" "TP21" (at 158.75 40.64 0)
       (effects (font (size 1.27 1.27)) (justify right))
     )
@@
     (instances
       (project "pico_synth_sandbox"
-        (path "/bfc01388-33ce-4b1a-9d2f-82d750172e5a"
-          (reference "TP12") (unit 1)
-        )
         (path "/bfc01388-33ce-4b1a-9d2f-82d750172e5a/c37b2c46-91dc-4067-923d-eccca1cbe357"
           (reference "TP21") (unit 1)
@@
   (symbol (lib_id "Connector:TestPoint") (at 172.72 50.8 0) (mirror y) (unit 1)
     (in_bom yes) (on_board yes) (dnp no)
-    (property "Reference" "TP14" (at 173.99 49.53 0)
+    (property "Reference" "TP23" (at 173.99 49.53 0)
       (effects (font (size 1.27 1.27)) (justify right))
     )
@@
     (instances
       (project "pico_synth_sandbox"
-        (path "/bfc01388-33ce-4b1a-9d2f-82d750172e5a"
-          (reference "TP14") (unit 1)
-        )
         (path "/bfc01388-33ce-4b1a-9d2f-82d750172e5a/c37b2c46-91dc-4067-923d-eccca1cbe357"
           (reference "TP23") (unit 1)
@@
   (symbol (lib_id "Connector:TestPoint") (at 142.24 41.91 0) (mirror y) (unit 1)
     (in_bom yes) (on_board yes) (dnp no)
-    (property "Reference" "TP10" (at 143.51 40.64 0)
+    (property "Reference" "TP19" (at 143.51 40.64 0)
       (effects (font (size 1.27 1.27)) (justify right))
     )
@@
     (instances
       (project "pico_synth_sandbox"
-        (path "/bfc01388-33ce-4b1a-9d2f-82d750172e5a"
-          (reference "TP10") (unit 1)
-        )
         (path "/bfc01388-33ce-4b1a-9d2f-82d750172e5a/c37b2c46-91dc-4067-923d-eccca1cbe357"
           (reference "TP19") (unit 1)
@@
   (symbol (lib_id "Connector:TestPoint") (at 119.38 50.8 0) (mirror y) (unit 1)
     (in_bom yes) (on_board yes) (dnp no)
-    (property "Reference" "TP7" (at 120.65 49.53 0)
+    (property "Reference" "TP16" (at 120.65 49.53 0)
       (effects (font (size 1.27 1.27)) (justify right))
     )
@@
     (instances
       (project "pico_synth_sandbox"
-        (path "/bfc01388-33ce-4b1a-9d2f-82d750172e5a"
-          (reference "TP7") (unit 1)
-        )
         (path "/bfc01388-33ce-4b1a-9d2f-82d750172e5a/c37b2c46-91dc-4067-923d-eccca1cbe357"
           (reference "TP16") (unit 1)
@@
   (symbol (lib_id "Connector:TestPoint") (at 88.9 41.91 0) (mirror y) (unit 1)
     (in_bom yes) (on_board yes) (dnp no)
-    (property "Reference" "TP3" (at 90.17 40.64 0)
+    (property "Reference" "TP12" (at 90.17 40.64 0)
       (effects (font (size 1.27 1.27)) (justify right))
     )
@@
     (instances
       (project "pico_synth_sandbox"
-        (path "/bfc01388-33ce-4b1a-9d2f-82d750172e5a"
-          (reference "TP3") (unit 1)
-        )
         (path "/bfc01388-33ce-4b1a-9d2f-82d750172e5a/c37b2c46-91dc-4067-923d-eccca1cbe357"
           (reference "TP12") (unit 1)
@@
   (symbol (lib_id "Connector:TestPoint") (at 104.14 41.91 0) (mirror y) (unit 1)
     (in_bom yes) (on_board yes) (dnp no)
-    (property "Reference" "TP5" (at 105.41 40.64 0)
+    (property "Reference" "TP14" (at 105.41 40.64 0)
       (effects (font (size 1.27 1.27)) (justify right))
     )
@@
     (instances
       (project "pico_synth_sandbox"
-        (path "/bfc01388-33ce-4b1a-9d2f-82d750172e5a"
-          (reference "TP5") (unit 1)
-        )
         (path "/bfc01388-33ce-4b1a-9d2f-82d750172e5a/c37b2c46-91dc-4067-923d-eccca1cbe357"
           (reference "TP14") (unit 1)
@@
   (symbol (lib_id "Connector:TestPoint") (at 81.28 50.8 0) (mirror y) (unit 1)
     (in_bom yes) (on_board yes) (dnp no)
-    (property "Reference" "TP2" (at 82.55 49.53 0)
+    (property "Reference" "TP11" (at 82.55 49.53 0)
       (effects (font (size 1.27 1.27)) (justify right))
     )
@@
     (instances
       (project "pico_synth_sandbox"
-        (path "/bfc01388-33ce-4b1a-9d2f-82d750172e5a"
-          (reference "TP2") (unit 1)
-        )
         (path "/bfc01388-33ce-4b1a-9d2f-82d750172e5a/c37b2c46-91dc-4067-923d-eccca1cbe357"
           (reference "TP11") (unit 1)
@@
   (symbol (lib_id "Connector:TestPoint") (at 96.52 50.8 0) (mirror y) (unit 1)
     (in_bom yes) (on_board yes) (dnp no)
-    (property "Reference" "TP4" (at 97.79 49.53 0)
+    (property "Reference" "TP13" (at 97.79 49.53 0)
       (effects (font (size 1.27 1.27)) (justify right))
     )
@@
     (instances
       (project "pico_synth_sandbox"
-        (path "/bfc01388-33ce-4b1a-9d2f-82d750172e5a"
-          (reference "TP4") (unit 1)
-        )
         (path "/bfc01388-33ce-4b1a-9d2f-82d750172e5a/c37b2c46-91dc-4067-923d-eccca1cbe357"
           (reference "TP13") (unit 1)
@@
   (symbol (lib_id "Connector:TestPoint") (at 73.66 50.8 0) (mirror y) (unit 1)
     (in_bom yes) (on_board yes) (dnp no)
-    (property "Reference" "TP1" (at 74.93 49.53 0)
+    (property "Reference" "TP10" (at 74.93 49.53 0)
       (effects (font (size 1.27 1.27)) (justify right))
     )
@@
     (instances
       (project "pico_synth_sandbox"
-        (path "/bfc01388-33ce-4b1a-9d2f-82d750172e5a"
-          (reference "TP1") (unit 1)
-        )
         (path "/bfc01388-33ce-4b1a-9d2f-82d750172e5a/c37b2c46-91dc-4067-923d-eccca1cbe357"
           (reference "TP10") (unit 1)
@@
   (symbol (lib_id "Connector:TestPoint") (at 134.62 50.8 0) (mirror y) (unit 1)
     (in_bom yes) (on_board yes) (dnp no)
-    (property "Reference" "TP9" (at 135.89 49.53 0)
+    (property "Reference" "TP18" (at 135.89 49.53 0)
       (effects (font (size 1.27 1.27)) (justify right))
     )
@@
     (instances
       (project "pico_synth_sandbox"
-        (path "/bfc01388-33ce-4b1a-9d2f-82d750172e5a"
-          (reference "TP9") (unit 1)
-        )
         (path "/bfc01388-33ce-4b1a-9d2f-82d750172e5a/c37b2c46-91dc-4067-923d-eccca1cbe357"
           (reference "TP18") (unit 1)
@@
   (symbol (lib_id "Connector:TestPoint") (at 187.96 50.8 0) (mirror y) (unit 1)
     (in_bom yes) (on_board yes) (dnp no)
-    (property "Reference" "TP16" (at 189.23 49.53 0)
+    (property "Reference" "TP25" (at 189.23 49.53 0)
       (effects (font (size 1.27 1.27)) (justify right))
     )
@@
     (instances
       (project "pico_synth_sandbox"
-        (path "/bfc01388-33ce-4b1a-9d2f-82d750172e5a"
-          (reference "TP16") (unit 1)
-        )
         (path "/bfc01388-33ce-4b1a-9d2f-82d750172e5a/c37b2c46-91dc-4067-923d-eccca1cbe357"
           (reference "TP25") (unit 1)
@@
   (symbol (lib_id "Connector:TestPoint") (at 127 41.91 0) (mirror y) (unit 1)
     (in_bom yes) (on_board yes) (dnp no)
-    (property "Reference" "TP8" (at 128.27 40.64 0)
+    (property "Reference" "TP17" (at 128.27 40.64 0)
       (effects (font (size 1.27 1.27)) (justify right))
     )
@@
     (instances
       (project "pico_synth_sandbox"
-        (path "/bfc01388-33ce-4b1a-9d2f-82d750172e5a"
-          (reference "TP8") (unit 1)
-        )
         (path "/bfc01388-33ce-4b1a-9d2f-82d750172e5a/c37b2c46-91dc-4067-923d-eccca1cbe357"
           (reference "TP17") (unit 1)
@@
   (symbol (lib_id "Connector:TestPoint") (at 111.76 50.8 0) (mirror y) (unit 1)
     (in_bom yes) (on_board yes) (dnp no)
-    (property "Reference" "TP6" (at 113.03 49.53 0)
+    (property "Reference" "TP15" (at 113.03 49.53 0)
       (effects (font (size 1.27 1.27)) (justify right))
     )
@@
     (instances
       (project "pico_synth_sandbox"
-        (path "/bfc01388-33ce-4b1a-9d2f-82d750172e5a"
-          (reference "TP6") (unit 1)
-        )
         (path "/bfc01388-33ce-4b1a-9d2f-82d750172e5a/c37b2c46-91dc-4067-923d-eccca1cbe357"
           (reference "TP15") (unit 1)
@@
   (symbol (lib_id "Connector:TestPoint") (at 180.34 41.91 0) (mirror y) (unit 1)
     (in_bom yes) (on_board yes) (dnp no)
-    (property "Reference" "TP15" (at 181.61 40.64 0)
+    (property "Reference" "TP24" (at 181.61 40.64 0)
       (effects (font (size 1.27 1.27)) (justify right))
     )
@@
     (instances
       (project "pico_synth_sandbox"
-        (path "/bfc01388-33ce-4b1a-9d2f-82d750172e5a"
-          (reference "TP15") (unit 1)
-        )
         (path "/bfc01388-33ce-4b1a-9d2f-82d750172e5a/c37b2c46-91dc-4067-923d-eccca1cbe357"
           (reference "TP24") (unit 1)
@@
   (symbol (lib_id "Connector:TestPoint") (at 165.1 50.8 0) (mirror y) (unit 1)
     (in_bom yes) (on_board yes) (dnp no)
-    (property "Reference" "TP13" (at 166.37 49.53 0)
+    (property "Reference" "TP22" (at 166.37 49.53 0)
       (effects (font (size 1.27 1.27)) (justify right))
     )
@@
     (instances
       (project "pico_synth_sandbox"
-        (path "/bfc01388-33ce-4b1a-9d2f-82d750172e5a"
-          (reference "TP13") (unit 1)
-        )
         (path "/bfc01388-33ce-4b1a-9d2f-82d750172e5a/c37b2c46-91dc-4067-923d-eccca1cbe357"
           (reference "TP22") (unit 1)

Commit message: Updated to KiCad 8.0 and fixed TTP229 3.3v net.
Connections:
- net +3V3 renamed +3.3V
