File: midi.kicad_sch (KiCad schematic)
At the start: 12 parts, among them J1 MIDIIN, J2 MIDIOUT, J3 MIDIIN, J3 MIDIOUT, U5 6N138

Commit message: Revision 2 of schematic and pcb.
Parts:
- removed C19, C20: 1uF, Capacitor_THT:CP_Radial_D5.0mm_P2.00mm, symbol Device:C_Polarized_Small
- removed D1: 1N914, Diode_THT:D_DO-35_SOD27_P7.62mm_Horizontal, symbol Diode:1N914
- removed J3: MIDIOUT, Connector_Audio:Jack_3.5mm_CUI_SJ1-3525N_Horizontal, symbol Connector_Audio:AudioJack3_SwitchTR
- removed J3: MIDIIN, Connector_Audio:Jack_3.5mm_CUI_SJ1-3525N_Horizontal, symbol Connector_Audio:AudioJack3_SwitchTR
- removed R27: 220, Resistor_THT:R_Axial_DIN0207_L6.3mm_D2.5mm_P7.62mm_Horizontal, symbol Device:R_Small
- removed R28: 4.7k, Resistor_THT:R_Axial_DIN0207_L6.3mm_D2.5mm_P7.62mm_Horizontal, symbol Device:R_Small
- removed R29: 470, Resistor_THT:R_Axial_DIN0207_L6.3mm_D2.5mm_P7.62mm_Horizontal, symbol Device:R_Small
- removed U5: 6N138, Package_DIP:DIP-8_W7.62mm_Socket_LongPads, symbol Isolator:6N138
- added C27 (x2): 1uF, Capacitor_SMD:C_0805_2012Metric_Pad1.18x1.45mm_HandSolder, symbol Device:C_Small
- added D3: 1N4148W, Diode_SMD:D_SOD-123, symbol Diode:1N4148W
- added D4: MIDIIN, LED_SMD:LED_0805_2012Metric_Pad1.15x1.40mm_HandSolder, symbol Device:LED
- added D5: MIDIOUT, LED_SMD:LED_0805_2012Metric_Pad1.15x1.40mm_HandSolder, symbol Device:LED
- added J10: MIDIOUT, pico_synth_sandbox:Jack_3.5mm_PJ327A_Horizontal, symbol Connector_Audio:AudioJack4_SwitchT1
- added J10: MIDIIN, pico_synth_sandbox:Jack_3.5mm_PJ327A_Horizontal, symbol Connector_Audio:AudioJack4_SwitchT1
- added R20: 220, Resistor_SMD:R_0805_2012Metric_Pad1.20x1.40mm_HandSolder, symbol Device:R_Small
- added R21: 470, Resistor_SMD:R_0805_2012Metric_Pad1.20x1.40mm_HandSolder, symbol Device:R_Small
- added R22, R23: 2.2k, Resistor_SMD:R_0805_2012Metric_Pad1.20x1.40mm_HandSolder, symbol Device:R_Small
- added R24: 10, Resistor_SMD:R_0805_2012Metric_Pad1.20x1.40mm_HandSolder, symbol Device:R_Small
- added U9: H11L1, Package_DIP:SMDIP-6_W7.62mm, symbol Isolator:H11L1
- J1: footprint LED_SMD:LED_0805_2012Metric_Pad1.15x1.40mm_HandSolder -> (none)
- R25: renamed from R30; footprint Resistor_THT:R_Axial_DIN0207_L6.3mm_D2.5mm_P7.62mm_Horizontal -> Resistor_SMD:R_0805_2012Metric_Pad1.20x1.40mm_HandSolder
Connections:
- net +3.3V: now also C27.1, C27.1, R21.1, R22.1, R23.1, U9.6
- net GND: now also C27.2, C27.2, J10.S, U9.5
- net at J2.4, R25.2: now also J10.R1
- net at J1.4: now also J10.R1, R20.2
- net at J1.2: now also J10.S
- net at J1.5: now also D3.2 (A), J10.T, U9.2
- net MIDITX: no longer names the net of J2.5
- net MIDITX: now also J10.T, R24.1
- new net: D4.2 (A), R22.2
- new net: D5.2 (A), R23.2
- new net: D3.1 (K), R20.1, U9.1
- new net UART_RX: D4.1 (K), R21.2, U9.4
- new net UART_TX: D5.1 (K), R24.2
Other:
- title: pico_synth_sandbox -> pico_synth_sandbox - MIDI Input & Output
- moved on the sheet: J1, J2, R25

Commit message: Various minor schematic updates.
Parts:
- renumbered C27 to C54, C27 to C55, J10 to J7, J1 to J8, J2 to J9
Changed lines of the file:
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@@
   (symbol (lib_id "Connector:DIN-5_180degree") (at 217.17 96.52 270) (unit 1)
     (in_bom yes) (on_board yes) (dnp no) (fields_autoplaced)
-    (property "Reference" "J2" (at 209.55 96.5201 0)
+    (property "Reference" "J9" (at 209.55 96.5201 0)
       (effects (font (size 1.27 1.27)))
     )
@@
     (instances
       (project "pico_synth_sandbox"
-        (path "/bfc01388-33ce-4b1a-9d2f-82d750172e5a"
-          (reference "J2") (unit 1)
-        )
         (path "/bfc01388-33ce-4b1a-9d2f-82d750172e5a/d4704e72-f661-4b84-847a-157c0240dc16"
           (reference "J9") (unit 1)
@@
   (symbol (lib_id "Device:C_Small") (at 139.7 91.44 0) (mirror y) (unit 1)
     (in_bom yes) (on_board yes) (dnp no) (fields_autoplaced)
-    (property "Reference" "C27" (at 142.24 90.1763 0)
+    (property "Reference" "C54" (at 142.24 90.1763 0)
       (effects (font (size 1.27 1.27)) (justify right))
     )
@@
     (instances
       (project "pico_synth_sandbox"
-        (path "/bfc01388-33ce-4b1a-9d2f-82d750172e5a/93632245-6c20-4ae6-b62e-7dbbebc316d1"
-          (reference "C27") (unit 1)
-        )
         (path "/bfc01388-33ce-4b1a-9d2f-82d750172e5a/d4704e72-f661-4b84-847a-157c0240dc16"
           (reference "C54") (unit 1)
@@
     (instances
       (project "pico_synth_sandbox"
-        (path "/bfc01388-33ce-4b1a-9d2f-82d750172e5a/93632245-6c20-4ae6-b62e-7dbbebc316d1"
+        (path "/bfc01388-33ce-4b1a-9d2f-82d750172e5a/d4704e72-f661-4b84-847a-157c0240dc16"
           (reference "J10") (unit 1)
         )
-        (path "/bfc01388-33ce-4b1a-9d2f-82d750172e5a/d4704e72-f661-4b84-847a-157c0240dc16"
-          (reference "J10") (unit 1)
-        )
       )
     )
@@
   (symbol (lib_id "power:+3.3V") (at 172.72 78.74 0) (unit 1)
     (in_bom yes) (on_board yes) (dnp no)
-    (property "Reference" "#PWR08" (at 172.72 82.55 0)
+    (property "Reference" "#PWR0135" (at 172.72 82.55 0)
       (effects (font (size 1.27 1.27)) hide)
     )
@@
     (instances
       (project "pico_synth_sandbox"
-        (path "/bfc01388-33ce-4b1a-9d2f-82d750172e5a"
-          (reference "#PWR08") (unit 1)
-        )
         (path "/bfc01388-33ce-4b1a-9d2f-82d750172e5a/d4704e72-f661-4b84-847a-157c0240dc16"
           (reference "#PWR0135") (unit 1)
@@
   (symbol (lib_id "power:+3.3V") (at 139.7 80.01 0) (unit 1)
     (in_bom yes) (on_board yes) (dnp no) (fields_autoplaced)
-    (property "Reference" "#PWR09" (at 139.7 83.82 0)
+    (property "Reference" "#PWR0133" (at 139.7 83.82 0)
       (effects (font (size 1.27 1.27)) hide)
     )
@@
     (instances
       (project "pico_synth_sandbox"
-        (path "/bfc01388-33ce-4b1a-9d2f-82d750172e5a"
-          (reference "#PWR09") (unit 1)
-        )
         (path "/bfc01388-33ce-4b1a-9d2f-82d750172e5a/d4704e72-f661-4b84-847a-157c0240dc16"
           (reference "#PWR0133") (unit 1)
@@
   (symbol (lib_id "power:+3.3V") (at 219.71 78.74 0) (unit 1)
     (in_bom yes) (on_board yes) (dnp no) (fields_autoplaced)
-    (property "Reference" "#PWR09" (at 219.71 82.55 0)
+    (property "Reference" "#PWR0138" (at 219.71 82.55 0)
       (effects (font (size 1.27 1.27)) hide)
     )
@@
     (instances
       (project "pico_synth_sandbox"
-        (path "/bfc01388-33ce-4b1a-9d2f-82d750172e5a"
-          (reference "#PWR09") (unit 1)
-        )
         (path "/bfc01388-33ce-4b1a-9d2f-82d750172e5a/d4704e72-f661-4b84-847a-157c0240dc16"
           (reference "#PWR0138") (unit 1)
@@
   (symbol (lib_id "Connector_Audio:AudioJack4_SwitchT1") (at 34.29 93.98 0) (unit 1)
     (in_bom yes) (on_board yes) (dnp no)
-    (property "Reference" "J10" (at 24.13 94.615 0)
+    (property "Reference" "J7" (at 24.13 94.615 0)
       (effects (font (size 1.27 1.27)) (justify right))
     )
@@
     (instances
       (project "pico_synth_sandbox"
-        (path "/bfc01388-33ce-4b1a-9d2f-82d750172e5a/93632245-6c20-4ae6-b62e-7dbbebc316d1"
-          (reference "J10") (unit 1)
-        )
         (path "/bfc01388-33ce-4b1a-9d2f-82d750172e5a/d4704e72-f661-4b84-847a-157c0240dc16"
           (reference "J7") (unit 1)
@@
   (symbol (lib_id "power:+3.3V") (at 116.84 80.01 0) (unit 1)
     (in_bom yes) (on_board yes) (dnp no) (fields_autoplaced)
-    (property "Reference" "#PWR09" (at 116.84 83.82 0)
+    (property "Reference" "#PWR0132" (at 116.84 83.82 0)
       (effects (font (size 1.27 1.27)) hide)
     )
@@
     (instances
       (project "pico_synth_sandbox"
-        (path "/bfc01388-33ce-4b1a-9d2f-82d750172e5a"
-          (reference "#PWR09") (unit 1)
-        )
         (path "/bfc01388-33ce-4b1a-9d2f-82d750172e5a/d4704e72-f661-4b84-847a-157c0240dc16"
           (reference "#PWR0132") (unit 1)
@@
   (symbol (lib_id "Connector:DIN-5_180degree") (at 55.88 95.25 90) (mirror x) (unit 1)
     (in_bom yes) (on_board yes) (dnp no) (fields_autoplaced)
-    (property "Reference" "J1" (at 63.5 95.2501 0)
+    (property "Reference" "J8" (at 63.5 95.2501 0)
       (effects (font (size 1.27 1.27)))
     )
@@
     (instances
       (project "pico_synth_sandbox"
-        (path "/bfc01388-33ce-4b1a-9d2f-82d750172e5a"
-          (reference "J1") (unit 1)
-        )
         (path "/bfc01388-33ce-4b1a-9d2f-82d750172e5a/d4704e72-f661-4b84-847a-157c0240dc16"
           (reference "J8") (unit 1)
@@
   (symbol (lib_id "power:+3.3V") (at 106.68 80.01 0) (unit 1)
     (in_bom yes) (on_board yes) (dnp no) (fields_autoplaced)
-    (property "Reference" "#PWR09" (at 106.68 83.82 0)
+    (property "Reference" "#PWR0131" (at 106.68 83.82 0)
       (effects (font (size 1.27 1.27)) hide)
     )
@@
     (instances
       (project "pico_synth_sandbox"
-        (path "/bfc01388-33ce-4b1a-9d2f-82d750172e5a"
-          (reference "#PWR09") (unit 1)
-        )
         (path "/bfc01388-33ce-4b1a-9d2f-82d750172e5a/d4704e72-f661-4b84-847a-157c0240dc16"
           (reference "#PWR0131") (unit 1)
@@
   (symbol (lib_id "Device:C_Small") (at 172.72 95.25 0) (mirror y) (unit 1)
     (in_bom yes) (on_board yes) (dnp no) (fields_autoplaced)
-    (property "Reference" "C27" (at 175.26 93.9863 0)
+    (property "Reference" "C55" (at 175.26 93.9863 0)
       (effects (font (size 1.27 1.27)) (justify right))
     )
@@
     (instances
       (project "pico_synth_sandbox"
-        (path "/bfc01388-33ce-4b1a-9d2f-82d750172e5a/93632245-6c20-4ae6-b62e-7dbbebc316d1"
-          (reference "C27") (unit 1)
-        )
         (path "/bfc01388-33ce-4b1a-9d2f-82d750172e5a/d4704e72-f661-4b84-847a-157c0240dc16"
           (reference "C55") (unit 1)
@@
   (symbol (lib_id "power:+3.3V") (at 91.44 80.01 0) (unit 1)
     (in_bom yes) (on_board yes) (dnp no) (fields_autoplaced)
-    (property "Reference" "#PWR09" (at 91.44 83.82 0)
+    (property "Reference" "#PWR0129" (at 91.44 83.82 0)
       (effects (font (size 1.27 1.27)) hide)
     )
@@
     (instances
       (project "pico_synth_sandbox"
-        (path "/bfc01388-33ce-4b1a-9d2f-82d750172e5a"
-          (reference "#PWR09") (unit 1)
-        )
         (path "/bfc01388-33ce-4b1a-9d2f-82d750172e5a/d4704e72-f661-4b84-847a-157c0240dc16"
           (reference "#PWR0129") (unit 1)
@@
   (symbol (lib_id "power:+3.3V") (at 196.85 78.74 0) (unit 1)
     (in_bom yes) (on_board yes) (dnp no) (fields_autoplaced)
-    (property "Reference" "#PWR09" (at 196.85 82.55 0)
+    (property "Reference" "#PWR0137" (at 196.85 82.55 0)
       (effects (font (size 1.27 1.27)) hide)
     )
@@
     (instances
       (project "pico_synth_sandbox"
-        (path "/bfc01388-33ce-4b1a-9d2f-82d750172e5a"
-          (reference "#PWR09") (unit 1)
-        )
         (path "/bfc01388-33ce-4b1a-9d2f-82d750172e5a/d4704e72-f661-4b84-847a-157c0240dc16"
           (reference "#PWR0137") (unit 1)
